File: hardware/kicad/msx-joyblue-v1/msx-joyblue.kicad_pcb (KiCad board)
At the start: 2 copper layers, 90 x 63 mm, 31 parts, among them J1 MSX PortA, J2 MSX PortB, J3 JOY PWR, J4 I2C, SW2 MODE, SW3 SWAP, U1 74LS05, U2 74LS05, U3 ESP32-DevKitC

Commit message: pcb: v1 build1
Signed-off-by: Albert Herranz <albert_herranz@yahoo.es>
Parts:
- U3: value ESP32-DevKitC -> ESP32 Kit; footprint Espressif:ESP32-DevKitC -> My_Components:X-NodeMCU-32-plus-ESP32-DevKitC
Routing:
- net GPIO_LED_J2: track 7.56 -> 13.0 mm
- net GND: track 29.9 -> 35.0 mm
- net GPIO_BOOTSTRAP_15_LED_J1: track 9.87 -> 14.9 mm
- net GPIO_LED_BT: track 11.3 -> 16.4 mm
- net I2C_SCL: track 13.6 -> 18.4 mm
- net I2C_SDA: track 15.2 -> 20.0 mm
- net GPIO_J2_UP: track 49.3 -> 51.9 mm
- net GPIO_J2_TRIG1: track 45.9 -> 48.5 mm
- net GPIO_J2_DOWN: track 53.6 -> 56.1 mm
- net unconnected-(U3-U0TXD/GPIO1-Pad35): track 0.00 -> 2.54 mm
- net unconnected-(U3-U0RXD/GPIO3-Pad34): track 0.00 -> 2.54 mm
- net unconnected-(U3-SD_DATA1/GPIO8-Pad22): track 0.00 -> 2.54 mm
- net unconnected-(U3-GPIO0/BOOT/ADC2_CH1-Pad25): track 0.00 -> 2.54 mm
- net GPIO_J2_TRIG2: track 50.1 -> 52.7 mm
- net GPIO_BOOTSTRAP_04: track 0.00 -> 2.54 mm
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Other:
- board text added: "msx-joyblue-v1 Build1"
- board text removed: "msx-joyblue-v1"

Commit message: pcb: v1 build1a
Signed-off-by: Albert Herranz <albert_herranz@yahoo.es>
Parts:
- added JP3: J1 Fuse Bypass, Connector_PinHeader_2.54mm:PinHeader_1x02_P2.54mm_Vertical, F.Cu at (117.2, 107.3)
- added JP4: J2 Fuse Bypass, Connector_PinHeader_2.54mm:PinHeader_1x02_P2.54mm_Vertical, F.Cu at (117.2, 79.4)
Routing:
- net /J2_PWR: track 25.2 -> 34.8 mm
- net /J1_PWR: track 25.2 -> 34.8 mm
Other:
- board text added: "msx-joyblue-v1 Build1a"
- board text removed: "msx-joyblue-v1 Build1"
