File: hardware/kicad/msx-joyblue-v1/msx-joyblue.kicad_sch (KiCad schematic)
At the start: 33 parts, among them J1 MSX PortA, J2 MSX PortB, J3 JOY PWR, J4 I2C, SW2 MODE, SW3 SWAP, U1 74LS05, U2 74LS05, U3 ESP32-DevKitC

Commit message: pcb: v1 build1a
Signed-off-by: Albert Herranz <albert_herranz@yahoo.es>
Parts:
- added JP3: J1 Fuse Bypass, Connector_PinHeader_2.54mm:PinHeader_1x02_P2.54mm_Vertical, symbol Jumper:Jumper_2_Open
- added JP4: J2 Fuse Bypass, Connector_PinHeader_2.54mm:PinHeader_1x02_P2.54mm_Vertical, symbol Jumper:Jumper_2_Open
- U3: value ESP32-DevKitC -> ESP32 Kit; footprint Espressif:ESP32-DevKitC -> My_Components:X-NodeMCU-32-plus-ESP32-DevKitC
Connections:
- net J1_PWR: now also JP3.1 (A)
- net J2_PWR: now also JP4.1 (A)
- net JOY_5V: now also JP3.2 (B), JP4.2 (B)
Other:
- moved on the sheet: D2, D3, D4, R1, R2, R3, R8, R9, SW2, SW3
